Commit message: Fix hand pose geometry: curl toward the palm, not straight up
Each finger's j1 joint mounted with no pitch, so q=0 pointed straight up
out of the palm's face and increasing q tipped it toward flat/horizontal —
paper and rock looked like an open spread hand and a flat hand respectively,
inverted from a real fist. Pitching the mount 90 degrees makes q=0 extend
forward (open hand) and larger q curl down into the palm (closing fist),
verified against the actual palm->fingertip TF for all three poses.

Found by testing with the real camera: RViz showed all three gestures and
held the last pose across a signal loss and a camera reconnect, but the
finger shapes didn't look right.

File: computer_vision/gesture_robot/ros2_ws/src/gesture_sim/urdf/simple_hand.urdf.xacro (robot description, xacro)
@@ -15,4 +15,10 @@
   <xacro:property name="finger_mass" value="0.02"/>
   <xacro:property name="joint_upper" value="1.6"/>
+  <!-- Segment geometry extends along its own local +Z. Pitching the j1
+       mount by 90 deg about Y makes q=0 point that +Z straight out along
+       the palm's +X (an open, extended finger); increasing q then curls it
+       toward -Z (down, into the palm), matching a closing fist. Without
+       this pitch, q=0 points straight up out of the palm's face instead. -->
+  <xacro:property name="finger_rest_pitch" value="1.5708"/>
   <material name="skin">
     <color rgba="0.87 0.72 0.60 1.0"/>
@@ -46,5 +52,5 @@
       <parent link="palm"/>
       <child link="${name}_proximal"/>
-      <origin xyz="${x} ${y} ${z}" rpy="0 0 ${yaw}"/>
+      <origin xyz="${x} ${y} ${z}" rpy="0 ${finger_rest_pitch} ${yaw}"/>
       <axis xyz="0 1 0"/>
       <limit lower="0.0" upper="${joint_upper}" effort="5.0" velocity="3.0"/>
