Commit message: Phase 4 (stage B, hand): run the hand in Gazebo Harmonic
The same hand model and controllers now run in Gazebo via gz_ros2_control
when use_gazebo:=true, driven by physics instead of mock hardware, with no
change to the model, controllers, or behavior node.

macOS/RoboStack fixes: add the conda lib dir to GZ_SIM_SYSTEM_PLUGIN_PATH so
the gz_ros2_control plugin loads, bridge the simulation /clock, and use RViz2
as the viewer since Gazebo's OGRE/Metal GUI does not render on macOS. Lift the
palm off the ground and set position_proportional_gain to 0.5 so the fingers
track their commanded poses instead of barely moving.

Also gitignore SESSION_NOTES.md. TurtleBot3 in Gazebo is a follow-up.

Co-Authored-By: Claude Opus 4.8 <noreply@anthropic.com>

File: computer_vision/gesture_robot/ros2_ws/src/gesture_sim/urdf/simple_hand.urdf.xacro (robot description, xacro)
@@ -77,7 +77,11 @@
   </xacro:macro>
   <link name="world"/>
+  <!-- Lift the palm off the ground so the fingers have room to curl down in
+       Gazebo without colliding with the ground plane (which pinned the curl in
+       RViz-free physics). Harmless in RViz. -->
   <joint name="world_to_palm" type="fixed">
     <parent link="world"/>
     <child link="palm"/>
+    <origin xyz="0 0 0.5" rpy="0 0 0"/>
   </joint>
   <link name="palm">
@@ -118,3 +122,19 @@
     <joint name="pinky_j2"><command_interface name="position"/><state_interface name="position"/></joint>
   </ros2_control>
+  <!-- In Gazebo, gz_ros2_control hosts the controller manager itself through
+       this plugin, so the launch file leaves out the standalone ros2_control_node
+       used in RViz-only (stage A). Inert unless use_gazebo:=true. -->
+  <xacro:if value="$(arg use_gazebo)">
+    <gazebo>
+      <plugin filename="gz_ros2_control-system"
+              name="gz_ros2_control::GazeboSimROS2ControlPlugin">
+        <parameters>$(find gesture_sim)/config/hand_controllers.yaml</parameters>
+        <!-- Position command interface drives joint velocity as
+             gain * position_error * update_rate. The 0.1 default barely moves
+             the fingers; 0.5 tracks the poses without the oscillation the docs
+             warn about above ~1.0. -->
+        <position_proportional_gain>0.5</position_proportional_gain>
+      </plugin>
+    </gazebo>
+  </xacro:if>
 </robot>
